Commit message: Remove the J5-blocking side plate, J6-motor sweep relief in the wrist drum (J5 free ±90°)

File: urdf/magarm.urdf (robot description, URDF)
Before this commit: robot magarm, 9 links, 8 joints
Links:
- link link4: mass 0.6634 -> 0.6543

Commit message: J1 and J2 on DM-JH17-101 harmonic motors: new base and shoulder housing, MuJoCo model
J1: new base with a ring for the JH17, the 6707 bearing is gone.
J2: the fork is replaced by a shoulder housing on the J1 output, the upper arm is bolted
to the motor flange beside it (43 mm from the J1 axis). J2 range 0..200 deg.
URDF, joint config and docs follow. sim/: MuJoCo model with the closed-chain gripper,
scene and pick-and-place demo. Logs are ignored.

File: urdf/magarm.urdf (robot description, URDF)
Before this commit: robot magarm, 9 links, 8 joints
Links:
- link base_link: mass 0.4974 -> 1.0768
- link link1: mass 0.0954 -> 1.1021
- link link2: mass 0.9443 -> 0.5877
Joints:
- joint joint1: limit lower=-2.79253 upper=2.79253 effort=27.0 velocity=5.8 -> lower=-2.79253 upper=2.79253 effort=54.0 velocity=3.14; origin xyz=0 0 0.06775 rpy=0 0 0 -> xyz=0 0 0.08275 rpy=0 0 0
- joint joint2: limit lower=0.0 upper=3.66519 effort=27.0 velocity=5.8 -> lower=0.0 upper=3.49066 effort=54.0 velocity=3.14; origin xyz=-0.0096 0 0.069 rpy=0 0 0 -> xyz=0 0.040875 0.054 rpy=0 0 0

Commit message: J2 as a fork with the JH17 inside the upper arm, bearing cheek on the other side; teleop handles removed
The J2 end of the upper arm becomes a drum for the motor, the fork holds the output flange and a 6705 on a
bolted-on cheek. J1 sits under the arm mid-plane, 61 mm below the J2 axis. J3 fold stop at 3.5 deg.
Sim: plate collision as a box, coarser motor meshes for the URDF.

File: urdf/magarm.urdf (robot description, URDF)
Before this commit: robot magarm, 9 links, 8 joints
Links:
- link link1: mass 1.1021 -> 0.1189
- link link2: mass 0.5877 -> 1.5728
- link link6: mass 0.4094 -> 0.3876
Joints:
- joint joint2: origin xyz=0 0.040875 0.054 rpy=0 0 0 -> xyz=0 0 0.061 rpy=0 0 0
- joint joint3: limit lower=-4.01426 upper=-0.0349 effort=27.0 velocity=5.8 -> lower=-4.01426 upper=-0.0611 effort=27.0 velocity=5.8
